File: eagle/Beagle_Buell Cape/motobone1.brd (EAGLE design)
At the start: 87.3 x 54.6 mm, 36 parts

Commit message: updates to Eagle PCB files
Parts:
- removed 12V_JACK: POWER_JACKPTH, SparkFun-Connectors:POWER_JACK_PTH
- removed HEAT: (no value), con-wago-500:W237-102
- removed R10, R11, R12, R13, R14, R15, R4, R5, R6, R7, R8, R9: 10k, SparkFun-Resistors:1206
- added J1: COMPUTER-PERIPHERAL-POWERRA, SparkFun-Connectors:COMPUTER-PERIPHERAL-POWER-RA
- moved U1 19.0 mm to (45.7, 12.7)
- moved PWR 17.8 mm to (21.6, 12.7)
- moved RST 16.5 mm to (34.3, 12.7)
- moved R2 12.7 mm to (26.7, 19.1)
- moved R1 11.4 mm to (34.3, 19.1)
- moved C1 10.0 mm to (62.9, 44.5), turned to 0 degrees
- moved R17 7.73 mm to (29.2, 45.7)
- moved R16 6.84 mm to (21.6, 45.7)
- moved CLOCK 6.35 mm to (54.6, 43.2)
- moved EEPROM 6.35 mm to (44.5, 43.2), turned to 270 degrees
- moved N_FET 2.84 mm to (24.1, 26.7)
- moved DC_REG 2.54 mm to (21.6, 38.1)
- moved DISPLAY 2.54 mm to (47.0, 33.0)
- moved ECU 2.54 mm to (47.0, 25.4)
- moved OXC 2.54 mm to (62.9, 41.3)
Connections:
- removed net N$13: HEAT.2, N_FET.S
- removed net N$14: R6.2, U$1.44
- removed net N$15: R4.2, U$1.42
- new net HEAT+: J1.5V, N_FET.S
- new net HEAT-: J1.GND, N_FET.D
- net 12V: now also J1.12V; no longer 12V_JACK.PWR
- net GND: now also J1.NC; no longer 12V_JACK.GND, 12V_JACK.GNDBREAK, R10.2, R11.1, R12.2, R13.2, R14.2, R4.1, R5.1, R6.1, R7.1, R8.1, R9.2, U$1.1, U$1.2, U$1.47, U$1.91, U$1.92
- net HEAT_GPIO: no longer R5.2
- net N$1: now also DISPLAY.4; no longer DISPLAY.2, R14.1
- net N$10: no longer R9.1
- net N$11: no longer R13.1
- net N$12: now also U$1.1, U$1.2, U$1.47, U$1.91, U$1.92; no longer HEAT.1, N_FET.D
- net N$2: no longer R7.2
- net N$22: no longer R11.2
- net N$3: now also DISPLAY.2; no longer DISPLAY.4, R12.1
- net N$4: no longer R15.2
- net N$7: no longer R8.2
- net N$9: no longer R10.1
- net PWR_BTN: now also DISPLAY.7
- net RST_BTN: now also DISPLAY.5
- net SYS_5V: no longer R15.1
Routing:
- net N$12: track 11.9 -> 150.6 mm
- net GND: track 265.6 -> 203.0 mm, vias 2 -> 1
- net N$9: track 47.1 -> 15.4 mm
- net VDD_3V3: track 81.9 -> 57.5 mm
- net N$4: track 41.2 -> 16.9 mm
- net N$2: track 35.9 -> 12.5 mm, vias 3 -> 0
- net N$10: track 31.8 -> 12.7 mm, vias 2 -> 1
- net N$26: track 6.51 -> 24.8 mm
- net N$3: track 37.1 -> 55.4 mm, vias 0 -> 2
- net N$15: track 18.2 -> 0.00 mm
- net N$25: track 9.57 -> 27.4 mm
- net N$1: track 32.4 -> 46.6 mm
- net N$23: track 21.1 -> 8.63 mm
- net N$13: track 10.8 -> 0.00 mm
- net N$14: track 10.7 -> 0.00 mm
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Other:
- board text added: "12V"
- board text added: "GND"
- board text added: "HEAT+"
- board text added: "HEAT-"
- board text added: "Logic Shifter"
- board text removed: "+"
- board text removed: "-"
- board text removed: "10k"
- board text removed: "HEAT"
