File: eagle/Beagle_Buell Cape/motobone1.sch (EAGLE design)
At the start: 36 parts

Commit message: updates to Eagle PCB files
Parts:
- removed 12V_JACK: POWER_JACKPTH, SparkFun-Connectors:POWER_JACKPTH
- removed HEAT: (no value), con-wago-500:W237-102
- removed R10, R11, R12, R13, R14, R15, R4, R5, R6, R7, R8, R9: 10k, SparkFun-Resistors:RESISTOR1206
- added J1: COMPUTER-PERIPHERAL-POWERRA, SparkFun-Connectors:COMPUTER-PERIPHERAL-POWERRA
Connections:
- removed net N$13: HEAT-2.KL, N_FET.S
- removed net N$14: R6.2, U$1.GPIO2_9
- removed net N$15: R4.2, U$1.GPIO2_11
- new net HEAT+: J1.5V, N_FET.S
- new net HEAT-: J1.GND, N_FET.D
- net 12V: now also J1.12V; no longer 12V_JACK.PWR
- net GND: now also J1.NC; no longer 12V_JACK.GND, 12V_JACK.GNDBREAK, R10.2, R11.1, R12.2, R13.2, R14.2, R4.1, R5.1, R6.1, R7.1, R8.1, R9.2
- net HEAT_GPIO: no longer R5.2
- net N$1: now also DISPLAY.4; no longer DISPLAY.2, R14.1
- net N$10: no longer R9.1
- net N$11: no longer R13.1
- net N$12: now also U$1.GND@1, U$1.GND@4, U$1.GND@6, U$1.GND@7, U$1.GND@8; no longer HEAT-1.KL, N_FET.D
- net N$2: no longer R7.2
- net N$22: no longer R11.2
- net N$3: now also DISPLAY.2; no longer DISPLAY.4, R12.1
- net N$4: no longer R15.2
- net N$7: no longer R8.2
- net N$9: no longer R10.1
- net PWR_BTN: now also DISPLAY.7
- net RST_BTN: now also DISPLAY.5
- net SYS_5V: no longer R15.1
Other:
- note added: "12v"
- note added: "GND"
- note added: "Heat+"
- note added: "Heat-"
