File: eagle/Motobone Cape SMD/motobone2.sch (EAGLE design)
At the start: 23 parts, among them J1 COMPUTER-PERIPHERAL-POWERRA

Commit message: updating Eagle files
Parts:
- removed C1: 0.1uF, SparkFun-Capacitors:10UF-6.3V-20%(1206)
- removed CLOCK: DS1307SO8, SparkFun-FreqCtrl:DS1307SO8
- removed EEPROM: EEPROM-I2CSMD, SparkFun-DigitalIC:EEPROM-I2CSMD
- removed OXC: (no value), crystal:CRYSTALTC38H
- added D1: (no value), SparkFun-DiscreteSemi:DIODE1N4148
- added IC3: DS3231/SO, adafruit:DS3231/SO
- added Q1: FQN1N50C, adafruit:FQN1N50C
- added R3: 10k, SparkFun-Resistors:RESISTOR1206
- added R4, R5: .1uf, SparkFun-Capacitors:10UF-TANT
- added U$2: LM3480IM4, SparkFun-PowerIC:LM3480IM4
- added U4: LS20126, SparkFun-RF:LS20126
- BAT1: value (none) -> 3v
- R16: value 10uf -> .33uf
- R17: value 10uf -> .1uf
- R2: value 3k -> 1k
- U1: value (none) -> EEPROM-I2CSMD; device SparkFun-DigitalIC:TXB0104PWRSOIC14 -> SparkFun-DigitalIC:EEPROM-I2CSMD
Connections:
- removed net N$23: ECU.1, U1.B1
- removed net N$8: BAT1.-, CLOCK.VBATT
- new net N$13: ECU.6, U$1.GPIO1_13
- new net N$14: ECU.8, U$1.EHRPWM2B
- new net N$16: U$1.UART1_RXD, U4.TX
- new net N$18: U$1.UART1_TXD, U4.RX
- net 12V: now also R4.+, U$2.IN
- net GND: now also BAT1.-, ECU.5, ECU.7, IC3.GND, IC3.NC, IC3.NC1, IC3.NC2, IC3.NC3, IC3.NC4, IC3.NC5, IC3.NC6, IC3.NC7, R3.1, R4.-, R5.-, U$1.GND@1, U$1.GND@4, U$1.GND@6, U$1.GND@7, U$1.GND@8, U$2.GND, U1.A0, U1.A1, U1.VSS, U1.WP, U4.GND@1, U4.GND@2, U4.GND@3; no longer BAT1.+, CLOCK.GND, EEPROM.A0, EEPROM.A1, EEPROM.A2, EEPROM.VSS, EEPROM.WP, U1.GND
- net N$10: now also U1.SDA; no longer EEPROM.SDA
- net N$12: now also Q1.G, U$1.UART5_TXD; no longer U$1.GND@1, U$1.GND@4, U$1.GND@6, U$1.GND@7, U$1.GND@8
- net N$17: now also U$1.AIN5; no longer U$1.GPIO2_13
- net N$2: now also IC3.SCL; no longer CLOCK.SCL
- net N$22: now also U$1.GPIO1_0; no longer U$1.GPIO1_17
- net N$24: now also D1.C; no longer U1.B2
- net N$25: now also D1.A, R3.2; no longer U1.A2
- net N$26: now also ECU.1, Q1.D; no longer U$1.UART5_TXD, U1.A1
- net N$5: now also BAT1.+, IC3.VBAT; no longer C1.2, CLOCK.X2, OXC.1
- net N$6: now also R5.+, U$2.OUT, U4.VSTBY; no longer C1.1, CLOCK.X1, OXC.2
- net N$7: now also IC3.SDA; no longer CLOCK.SDA
- net N$9: now also U1.SCL; no longer EEPROM.SCL
- net SYS_5V: now also Q1.S; no longer CLOCK.VCC, EEPROM.VCC, U1.VCCB
- net VDD_3V3: now also IC3.VCC, U1.A2, U1.VCC, U4.EN, U4.VCC; no longer U1.VCCA
Other:
- moved on the sheet: BAT1
